File: Preamp/_autosave-AnywhereAmps_Preamp.kicad_pcb (KiCad board)
At the start: 2 copper layers, 69.1 x 45.2 mm, 59 parts, among them J1 +9V, J2 Battery, J3 VCC, J4 Switch, J5 Pwr LED, J6 POTI, J7 Audio_In, J8 Audio_Out, U1 PTPSM5601R5H, U2 MAX17562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

Commit message: - update pullup for 9V supply: Now, barrel GND is outer. - fix review findings (track spacing)
Other:
- board text added: "33n MLCC C10, C11, C12, C13, C14, C17 4.7u low ESR Tantalum C1, C2, C3, C6, C7, C8, C9, C15, C16 47u low ESR Tantalum C4, C5 390k R1, R7, R14 10k R2, R3, R4, R5, R6, R12, R15, R16, R17, R18, R19, R20, R21, R22 1.25k R8, R9, R10, R11, R13"
- board text removed: "33n MLCC C10, C11, C12, C13, C14, C17 4.7u low ESR Tantalum C1, C2, C3, C6, C7, C8, C9, C15, C16 47u low ESR Tantalum C4, C5 390k R1, R7, R9, R15 10k R2, R3, R4, R5, R6, R13, R16, R17, R18, R19, R20, R21, R22, R23 1.25k R8, R10, R11, R12, R14"
Changed lines of the file:
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@@
     )
   )
-  (gr_text "33n MLCC C10, C11, C12, C13, C14, C17\n4.7u low ESR Tantalum C1, C2, C3, C6, C7, C8, C9, C15, C16\n47u low ESR Tantalum C4, C5\n390k R1, R7, R9, R15\n10k R2, R3, R4, R5, R6, R13, R16, R17, R18, R19, R20, R21, R22, R23\n1.25k R8, R10, R11, R12, R14" (at 169.418 116.586) (layer B.SilkS)
+  (gr_text "33n MLCC C10, C11, C12, C13, C14, C17\n4.7u low ESR Tantalum C1, C2, C3, C6, C7, C8, C9, C15, C16\n47u low ESR Tantalum C4, C5\n390k R1, R7, R14\n10k R2, R3, R4, R5, R6, R12, R15, R16, R17, R18, R19, R20, R21, R22\n1.25k R8, R9, R10, R11, R13" (at 169.418 116.586) (layer B.SilkS)
     (effects (font (size 0.8 0.8) (thickness 0.1)) (justify left mirror))
   )
@@
   (segment (start 112.014 124.968) (end 112.014 124.968) (width 1.65) (layer Front) (net 2))
   (segment (start 112.014 124.968) (end 112.014 124.968) (width 1.65) (layer Front) (net 2))
-  (via (at 112.014 124.968) (size 0.8) (drill 0.4) (layers Front Back) (net 2))
+  (via (at 112.014 124.968) (size 0.8) (drill 0.4) (layers Front Back) (net 2) (status 1000000))
   (segment (start 114.046 124.968) (end 112.014 124.968) (width 1.65) (layer Front) (net 2))
   (via (at 114.046 124.968) (size 0.8) (drill 0.4) (layers Front Back) (net 2))
