File: Preamp/AnywhereAmps_Preamp.sch (KiCad schematic (older format))
At the start: 57 parts, among them J1 +9V, J2 Battery, J3 VCC, J4 Switch, J5 Pwr LED, J6 POTI, J7 Audio_In, J8 Audio_Out, U1 PTPSM5601R5H, U2 MAX17562, U3 NE5532, U4 NE5532

Commit message: - switch to polarized capacitors for audio input - increase cap size for bypass on 9V rail - add polarity indicator on silk screen
Parts:
- removed C1, C14, C15, C2, C3, C6, C7, C8, C9: 4.7u, Capacitor_SMD:C_0805_2012Metric_Pad1.18x1.45mm_HandSolder, symbol Device:C
- removed C4, C5: 22u, Capacitor_SMD:C_0805_2012Metric_Pad1.18x1.45mm_HandSolder, symbol Device:C
- added C1, C15, C16, C2, C3, C6, C7, C8, C9: 4.7u, Capacitor_SMD:C_0805_2012Metric_Pad1.18x1.45mm_HandSolder, symbol Device:CP
- added C4, C5: 47u, Capacitor_SMD:C_1206_3216Metric_Pad1.33x1.80mm_HandSolder, symbol Device:CP
- renumbered C16 to C14

Commit message: - move VCC track away from M4 hole - exchange 383k resistors by E12 390k - use 10k resistors for VGND providers (quicker startup)
Parts:
- R1, R15, R7, R9: value 383k -> 390k
- R16, R17: value 383k -> 10k
Changed lines of the file:
@@
 P 950 1900
 F 0 "R1" H 880 1854 50  0000 R CNN
-F 1 "383k" H 880 1945 50  0000 R CNN
+F 1 "390k" H 880 1945 50  0000 R CNN
 F 2 "Resistor_SMD:R_0805_2012Metric_Pad1.20x1.40mm_HandSolder" V 880 1900 50  0001 C CNN
 F 3 "~" H 950 1900 50  0001 C CNN
@@
 P 5100 2050
 F 0 "R15" H 5030 2004 50  0000 R CNN
-F 1 "383k" H 5030 2095 50  0000 R CNN
+F 1 "390k" H 5030 2095 50  0000 R CNN
 F 2 "Resistor_SMD:R_0805_2012Metric_Pad1.20x1.40mm_HandSolder" V 5030 2050 50  0001 C CNN
 F 3 "~" H 5100 2050 50  0001 C CNN
@@
 P 6000 2700
 F 0 "R17" H 5930 2654 50  0000 R CNN
-F 1 "383k" H 5930 2745 50  0000 R CNN
+F 1 "10k" H 5930 2745 50  0000 R CNN
 F 2 "Resistor_SMD:R_0805_2012Metric_Pad1.20x1.40mm_HandSolder" V 5930 2700 50  0001 C CNN
 F 3 "~" H 6000 2700 50  0001 C CNN
@@
 P 6000 2300
 F 0 "R16" H 5930 2254 50  0000 R CNN
-F 1 "383k" H 5930 2345 50  0000 R CNN
+F 1 "10k" H 5930 2345 50  0000 R CNN
 F 2 "Resistor_SMD:R_0805_2012Metric_Pad1.20x1.40mm_HandSolder" V 5930 2300 50  0001 C CNN
 F 3 "~" H 6000 2300 50  0001 C CNN
@@
 P 1250 5950
 F 0 "R7" H 1180 5904 50  0000 R CNN
-F 1 "383k" H 1180 5995 50  0000 R CNN
+F 1 "390k" H 1180 5995 50  0000 R CNN
 F 2 "Resistor_SMD:R_0805_2012Metric_Pad1.20x1.40mm_HandSolder" V 1180 5950 50  0001 C CNN
 F 3 "~" H 1250 5950 50  0001 C CNN
@@
 P 3600 5550
 F 0 "R9" H 3530 5504 50  0000 R CNN
-F 1 "383k" H 3530 5595 50  0000 R CNN
+F 1 "390k" H 3530 5595 50  0000 R CNN
 F 2 "Resistor_SMD:R_0805_2012Metric_Pad1.20x1.40mm_HandSolder" V 3530 5550 50  0001 C CNN
 F 3 "~" H 3600 5550 50  0001 C CNN

Commit message: - update pullup for 9V supply: Now, barrel GND is outer. - fix review findings (track spacing)
Parts:
- removed R9: 390k, Resistor_SMD:R_0805_2012Metric_Pad1.20x1.40mm_HandSolder, symbol Device:R
- renumbered R11 to R10, R12 to R11, R13 to R12, R14 to R13, R15 to R14, R16 to R15, R17 to R16, R18 to R17, R19 to R18, R20 to R19, R21 to R20, R22 to R21, R23 to R22, R10 to R9
Connections:
- wire segments 189 -> 185
Other:
- note added: "Barrel Jack to disconnect GND and EN (NC switch). \nPullup to VCC then activates regulator."
- note removed: "Barrel Jack to connect +9V and EN (NO switch). \nPullup to VCC then activates regulator."

Commit message: - Change from EH to XH connectors, vertical - Re-align and place connectors - Delete LED, use TestPoint instead - Optimize 2mm tracks for shortness - update BOM
Parts:
- removed D1: Fault, LED_SMD:LED_0805_2012Metric_Pad1.15x1.40mm_HandSolder, symbol Device:LED
- added TP1: *Fault, TestPoint:TestPoint_Pad_D1.5mm, symbol Connector:TestPoint
- C4, C5: footprint Capacitor_SMD:C_1206_3216Metric_Pad1.33x1.80mm_HandSolder -> Capacitor_SMD:C_1210_3225Metric_Pad1.33x2.70mm_HandSolder
- J1, J8: footprint Connector_JST:JST_EH_S3B-EH_1x03_P2.50mm_Horizontal -> Connector_JST:JST_XH_B3B-XH-A_1x03_P2.50mm_Vertical
- J2, J3, J4, J5, J6, J7: footprint Connector_JST:JST_EH_S2B-EH_1x02_P2.50mm_Horizontal -> Connector_JST:JST_XH_B2B-XH-A_1x02_P2.50mm_Vertical
- R1, R14, R7: order https://www.mouser.de/ProductDetail/Panasonic/ERJ-6ENF3833V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 -> https://www.mouser.de/ProductDetail/KOA-Speer/RK73H2ATTD390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
- R11: order https://www.mouser.de/ProductDetail/Vishay-Dale/CRCW080510K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 -> https://www.mouser.de/ProductDetail/Panasonic/ERJ-6ENF1201V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
- R8: value 1.25k -> 390k
- U3: order (none) -> https://www.mouser.de/ProductDetail/Texas-Instruments/NE553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
- renumbered TP1 to TP2
Changed lines of the file:
@@
 F 2 "Resistor_SMD:R_0805_2012Metric_Pad1.20x1.40mm_HandSolder" V 880 1900 50  0001 C CNN
 F 3 "~" H 950 1900 50  0001 C CNN
-F 4 "https://www.mouser.de/ProductDetail/Panasonic/ERJ-6ENF3833V?qs=sGAEpiMZZMukHu%252BjC5l7Ye7G6YqZYGWLO48n8uKSaLY%3D" H 950 1900 50  0001 C CNN "order"
+F 4 "https://www.mouser.de/ProductDetail/KOA-Speer/RK73H2ATTD3903F?qs=D8YA4XSfdnQ%2FP3dwrcS24A%3D%3D" H 950 1900 50  0001 C CNN "order"
 	1    950  1900
 	-1   0    0    1
@@
 Wire Wire Line
 	4150 2100 4300 2100
-$Comp
-L Device:LED D1
-U 1 1 6150F2A0
-P 3100 3100
-F 0 "D1" V 3139 2982 50  0000 R CNN
-F 1 "Fault" V 3048 2982 50  0000 R CNN
-F 2 "LED_SMD:LED_0805_2012Metric_Pad1.15x1.40mm_HandSolder" H 3100 3100 50  0001 C CNN
-F 3 "~" H 3100 3100 50  0001 C CNN
-	1    3100 3100
-	0    -1   -1   0
-$EndComp
 Wire Wire Line
 	3100 2850 3100 2950
-Wire Wire Line
-	3100 3250 3100 3350
-Wire Wire Line
-	3100 3650 3100 3850
 $Comp
 L Connector:Conn_01x02_Male J4
@@
 F 0 "J4" H 3408 1031 50  0000 C CNN
 F 1 "Switch" H 3408 940 50  0000 C CNN
-F 2 "Connector_JST:JST_EH_S2B-EH_1x02_P2.50mm_Horizontal" H 3300 850 50  0001 C CNN
+F 2 "Connector_JST:JST_XH_B2B-XH-A_1x02_P2.50mm_Vertical" H 3300 850 50  0001 C CNN
 F 3 "~" H 3300 850 50  0001 C CNN
 	1    3300 850
@@
 F 0 "J3" H 2358 1031 50  0000 C CNN
 F 1 "VCC" H 2358 940 50  0000 C CNN
-F 2 "Connector_JST:JST_EH_S2B-EH_1x02_P2.50mm_Horizontal" H 2250 850 50  0001 C CNN
+F 2 "Connector_JST:JST_XH_B2B-XH-A_1x02_P2.50mm_Vertical" H 2250 850 50  0001 C CNN
 F 3 "~" H 2250 850 50  0001 C CNN
 	1    2250 850
@@
 L power:GND #PWR04
 U 1 1 61603409
+P 1100 4850
+F 0 "#PWR04" H 1100 4600 50  0001 C CNN
+F 1 "GND" V 1105 4722 50  0000 R CNN
+F 2 "" H 1100 4850 50  0001 C CNN
+F 3 "" H 1100 4850 50  0001 C CNN
+	1    1100 4850
+	0    -1   -1   0
+$EndComp
+$Comp
+L power:+9V #PWR03
+U 1 1 61605088
 P 1100 4750
-F 0 "#PWR04" H 1100 4500 50  0001 C CNN
-F 1 "GND" V 1105 4622 50  0000 R CNN
+F 0 "#PWR03" H 1100 4600 50  0001 C CNN
+F 1 "+9V" V 1115 4878 50  0000 L CNN
 F 2 "" H 1100 4750 50  0001 C CNN
 F 3 "" H 1100 4750 50  0001 C CNN
 	1    1100 4750
-	0    -1   -1   0
-$EndComp
-$Comp
-L power:+9V #PWR03
-U 1 1 61605088
-P 1100 4650
-F 0 "#PWR03" H 1100 4500 50  0001 C CNN
-F 1 "+9V" V 1115 4778 50  0000 L CNN
-F 2 "" H 1100 4650 50  0001 C CNN
-F 3 "" H 1100 4650 50  0001 C CNN
-	1    1100 4650
 	0    1    1    0
 $EndComp
@@
 F 2 "Resistor_SMD:R_0805_2012Metric_Pad1.20x1.40mm_HandSolder" V 5030 2050 50  0001 C CNN
 F 3 "~" H 5100 2050 50  0001 C CNN
-F 4 "https://www.mouser.de/ProductDetail/Panasonic/ERJ-6ENF3833V?qs=sGAEpiMZZMukHu%252BjC5l7Ye7G6YqZYGWLO48n8uKSaLY%3D" H 5100 2050 50  0001 C CNN "order"
+F 4 "https://www.mouser.de/ProductDetail/KOA-Speer/RK73H2ATTD3903F?qs=D8YA4XSfdnQ%2FP3dwrcS24A%3D%3D" H 5100 2050 50  0001 C CNN "order"
 	1    5100 2050
 	-1   0    0    1
@@
 F 0 "J5" H 4408 1031 50  0000 C CNN
 F 1 "Pwr LED" H 4408 940 50  0000 C CNN
-F 2 "Connector_JST:JST_EH_S2B-EH_1x02_P2.50mm_Horizontal" H 4300 850 50  0001 C CNN
+F 2 "Connector_JST:JST_XH_B2B-XH-A_1x02_P2.50mm_Vertical" H 4300 850 50  0001 C CNN
 F 3 "~" H 4300 850 50  0001 C CNN
 	1    4300 850
@@
 $EndComp
 $Comp
-L power:VCC #PWR023
+L power:VCC #PWR024
 U 1 1 616A4E71
+P 4950 950
+F 0 "#PWR024" H 4950 800 50  0001 C CNN
+F 1 "VCC" V 4965 1078 50  0000 L CNN
+F 2 "" H 4950 950 50  0001 C CNN
+F 3 "" H 4950 950 50  0001 C CNN
+	1    4950 950
+	0    1    1    0
+$EndComp
+$Comp
+L Device:R R11
+U 1 1 616A8084
+P 4650 850
+F 0 "R11" V 4750 850 50  0000 C CNN
+F 1 "1.25k" V 4850 850 50  0000 C CNN
+F 2 "Resistor_SMD:R_0805_2012Metric_Pad1.20x1.40mm_HandSolder" V 4580 850 50  0001 C CNN
+F 3 "~" H 4650 850 50  0001 C CNN
+F 4 "https://www.mouser.de/ProductDetail/Panasonic/ERJ-6ENF1201V?qs=sGAEpiMZZMtG0KNrPCHnjTg0x5DoQJ5PdamLOtzjzkA%3D" H 4650 850 50  0001 C CNN "order"
+	1    4650 850
+	0    1    1    0
+$EndComp
+$Comp
+L power:GND #PWR023
+U 1 1 616ABB8E
 P 4950 850
-F 0 "#PWR023" H 4950 700 50  0001 C CNN
-F 1 "VCC" V 4965 978 50  0000 L CNN
+F 0 "#PWR023" H 4950 600 50  0001 C CNN
+F 1 "GND" V 4955 722 50  0000 R CNN
 F 2 "" H 4950 850 50  0001 C CNN
 F 3 "" H 4950 850 50  0001 C CNN
 	1    4950 850
-	0    1    1    0
-$EndComp
-$Comp
-L Device:R R11
-U 1 1 616A8084
-P 4650 950
-F 0 "R11" V 4750 950 50  0000 C CNN
-F 1 "1.25k" V 4850 950 50  0000 C CNN
-F 2 "Resistor_SMD:R_0805_2012Metric_Pad1.20x1.40mm_HandSolder" V 4580 950 50  0001 C CNN
-F 3 "~" H 4650 950 50  0001 C CNN
-F 4 "https://www.mouser.de/ProductDetail/Vishay-Dale/CRCW080510K0FKEAC?qs=sGAEpiMZZMukHu%252BjC5l7Yc9NSHzGyJyzws8eSaD%252BBHw%3D" H 4650 950 50  0001 C CNN "order"
-	1    4650 950
-	0    1    1    0
-$EndComp
-Wire Wire Line
-	4500 850  4950 850
-$Comp
-L power:GND #PWR024
-U 1 1 616ABB8E
-P 4950 950
-F 0 "#PWR024" H 4950 700 50  0001 C CNN
-F 1 "GND" V 4955 822 50  0000 R CNN
-F 2 "" H 4950 950 50  0001 C CNN
-F 3 "" H 4950 950 50  0001 C CNN
-	1    4950 950
 	0    -1   -1   0
 $EndComp
 Wire Wire Line
-	4950 950  4800 950
+	4950 850  4800 850
 $Comp
 L Connector:Conn_01x02_Male J2
@@
 F 0 "J2" H 1008 1031 50  0000 C CNN
 F 1 "Battery" H 1008 940 50  0000 C CNN
-F 2 "Connector_JST:JST_EH_S2B-EH_1x02_P2.50mm_Horizontal" H 900 850 50  0001 C CNN
+F 2 "Connector_JST:JST_XH_B2B-XH-A_1x02_P2.50mm_Vertical" H 900 850 50  0001 C CNN
 F 3 "~" H 900 850 50  0001 C CNN
 	1    900  850
@@
 F 2 "Package_SO:SO-8_5.3x6.2mm_P1.27mm" H 7050 2600 50  0001 C CNN
 F 3 "http://www.ti.com/lit/ds/symlink/ne5532.pdf" H 7050 2600 50  0001 C CNN
+F 4 "https://www.mouser.de/ProductDetail/Texas-Instruments/NE5532APSR?qs=Tv815z3GeNT4dhpqaaa6LA%3D%3D" H 7050 2600 50  0001 C CNN "order"
 	2    7050 2600
 	1    0    0    -1
@@
 F 0 "J6" H 6058 1031 50  0000 C CNN
 F 1 "POTI" H 6058 940 50  0000 C CNN
-F 2 "Connector_JST:JST_EH_S2B-EH_1x02_P2.50mm_Horizontal" H 5950 850 50  0001 C CNN
+F 2 "Connector_JST:JST_XH_B2B-XH-A_1x02_P2.50mm_Vertical" H 5950 850 50  0001 C CNN
 F 3 "~" H 5950 850 50  0001 C CNN
 	1    5950 850
@@
 F 0 "J7" H 7158 1031 50  0000 C CNN
 F 1 "Audio_In" H 7158 940 50  0000 C CNN
-F 2 "Connector_JST:JST_EH_S2B-EH_1x02_P2.50mm_Horizontal" H 7050 850 50  0001 C CNN
+F 2 "Connector_JST:JST_XH_B2B-XH-A_1x02_P2.50mm_Vertical" H 7050 850 50  0001 C CNN
 F 3 "~" H 7050 850 50  0001 C CNN
 	1    7050 850
@@
 L Device:R R8
 U 1 1 6150D0F0
-P 3100 3500
-F 0 "R8" H 3170 3546 50  0000 L CNN
-F 1 "1.25k" H 3170 3455 50  0000 L CNN
-F 2 "Resistor_SMD:R_0805_2012Metric_Pad1.20x1.40mm_HandSolder" V 3030 3500 50  0001 C CNN
-F 3 "~" H 3100 3500 50  0001 C CNN
-F 4 "https://www.mouser.de/ProductDetail/Vishay-Dale/CRCW080510K0FKEAC?qs=sGAEpiMZZMukHu%252BjC5l7Yc9NSHzGyJyzws8eSaD%252BBHw%3D" H 3100 3500 50  0001 C CNN "order"
-	1    3100 3500
+P 3100 3100
+F 0 "R8" H 3170 3146 50  0000 L CNN
+F 1 "390k" H 3170 3055 50  0000 L CNN
+F 2 "Resistor_SMD:R_0805_2012Metric_Pad1.20x1.40mm_HandSolder" V 3030 3100 50  0001 C CNN
+F 3 "~" H 3100 3100 50  0001 C CNN
+F 4 "https://www.mouser.de/ProductDetail/Vishay-Dale/CRCW080510K0FKEAC?qs=sGAEpiMZZMukHu%252BjC5l7Yc9NSHzGyJyzws8eSaD%252BBHw%3D" H 3100 3100 50  0001 C CNN "order"
+	1    3100 3100
 	1    0    0    -1
 $EndComp
@@
 F 2 "Resistor_SMD:R_0805_2012Metric_Pad1.20x1.40mm_HandSolder" V 1180 5550 50  0001 C CNN
 F 3 "~" H 1250 5550 50  0001 C CNN
-F 4 "https://www.mouser.de/ProductDetail/Panasonic/ERJ-6ENF3833V?qs=sGAEpiMZZMukHu%252BjC5l7Ye7G6YqZYGWLO48n8uKSaLY%3D" H 1250 5550 50  0001 C CNN "order"
+F 4 "https://www.mouser.de/ProductDetail/KOA-Speer/RK73H2ATTD3903F?qs=D8YA4XSfdnQ%2FP3dwrcS24A%3D%3D" H 1250 5550 50  0001 C CNN "order"
 	1    1250 5550
 	-1   0    0    1
@@
 F 0 "J1" H 800 5050 50  0000 C CNN
 F 1 "+9V" H 800 4950 50  0000 C CNN
-F 2 "Connector_JST:JST_EH_S3B-EH_1x03_P2.50mm_Horizontal" H 750 4750 50  0001 C CNN
+F 2 "Connector_JST:JST_XH_B3B-XH-A_1x03_P2.50mm_Vertical" H 750 4750 50  0001 C CNN
 F 3 "~" H 750 4750 50  0001 C CNN
 	1    750  4750
 	1    0    0    -1
 $EndComp
-Text GLabel 1100 4850 2    50   Input ~ 0
+Text GLabel 1100 4650 2    50   Input ~ 0
 EN
 Wire Wire Line
@@
 F 0 "J8" H 8158 1081 50  0000 C CNN
 F 1 "Audio_Out" H 8158 990 50  0000 C CNN
-F 2 "Connector_JST:JST_EH_S3B-EH_1x03_P2.50mm_Horizontal" H 8050 900 50  0001 C CNN
+F 2 "Connector_JST:JST_XH_B3B-XH-A_1x03_P2.50mm_Vertical" H 8050 900 50  0001 C CNN
 F 3 "~" H 8050 900 50  0001 C CNN
 	1    8050 900
@@
 	8200 5800 8300 5800
 $Comp
-L Connector:TestPoint TP1
+L Connector:TestPoint TP2
 U 1 1 6206867A
 P 8300 5800
-F 0 "TP1" V 8254 5988 50  0000 L CNN
+F 0 "TP2" V 8254 5988 50  0000 L CNN
 F 1 "TestPoint" V 8345 5988 50  0000 L CNN
 F 2 "TestPoint:TestPoint_Pad_D1.5mm" H 8500 5800 50  0001 C CNN
@@
 F 0 "C4" H 3832 5504 50  0000 R CNN
 F 1 "47u" H 3832 5595 50  0000 R CNN
-F 2 "Capacitor_SMD:C_1206_3216Metric_Pad1.33x1.80mm_HandSolder" H 3988 5400 50  0001 C CNN
+F 2 "Capacitor_SMD:C_1210_3225Metric_Pad1.33x2.70mm_HandSolder" H 3988 5400 50  0001 C CNN
 F 3 "https://www.mouser.de/ProductDetail/AVX/TCNT476M016R0200A?qs=sGAEpiMZZMsh%252B1woXyUXj8cbwg7mY%252Bp%2FsXJ5jiWGcvo%3D" H 3950 5550 50  0001 C CNN
 	1    3950 5550
@@
 F 0 "C5" H 4068 6096 50  0000 L CNN
 F 1 "47u" H 4068 6005 50  0000 L CNN
-F 2 "Capacitor_SMD:C_1206_3216Metric_Pad1.33x1.80mm_HandSolder" H 3988 5900 50  0001 C CNN
+F 2 "Capacitor_SMD:C_1210_3225Metric_Pad1.33x2.70mm_HandSolder" H 3988 5900 50  0001 C CNN
 F 3 "https://www.mouser.de/ProductDetail/AVX/TCNT476M016R0200A?qs=sGAEpiMZZMsh%252B1woXyUXj8cbwg7mY%252Bp%2FsXJ5jiWGcvo%3D" H 3950 6050 50  0001 C CNN
 	1    3950 6050
@@
 Wire Wire Line
 	3450 5800 3950 5800
+Wire Wire Line
+	4950 950  4500 950
+$Comp
+L Connector:TestPoint TP1
+U 1 1 6185DB4A
+P 3100 3550
+F 0 "TP1" V 3054 3738 50  0000 L CNN
+F 1 "*Fault" V 3145 3738 50  0000 L CNN
+F 2 "TestPoint:TestPoint_Pad_D1.5mm" H 3300 3550 50  0001 C CNN
+F 3 "~" H 3300 3550 50  0001 C CNN
+	1    3100 3550
+	0    -1   -1   0
+$EndComp
+Connection ~ 3100 3550
+Wire Wire Line
+	3100 3550 3100 3850
+Wire Wire Line
+	3100 3250 3100 3550
 $EndSCHEMATC

Commit message: - fine-tune component placement - add batt and VCC copper layers - update SilkScreen
Changed lines of the file:
@@
 L power:VCC #PWR024
 U 1 1 616A4E71
+P 4950 850
+F 0 "#PWR024" H 4950 700 50  0001 C CNN
+F 1 "VCC" V 4965 978 50  0000 L CNN
+F 2 "" H 4950 850 50  0001 C CNN
+F 3 "" H 4950 850 50  0001 C CNN
+	1    4950 850
+	0    1    1    0
+$EndComp
+$Comp
+L power:GND #PWR023
+U 1 1 616ABB8E
 P 4950 950
-F 0 "#PWR024" H 4950 800 50  0001 C CNN
-F 1 "VCC" V 4965 1078 50  0000 L CNN
+F 0 "#PWR023" H 4950 700 50  0001 C CNN
+F 1 "GND" V 4955 822 50  0000 R CNN
 F 2 "" H 4950 950 50  0001 C CNN
 F 3 "" H 4950 950 50  0001 C CNN
 	1    4950 950
-	0    1    1    0
-$EndComp
-$Comp
-L Device:R R11
-U 1 1 616A8084
-P 4650 850
-F 0 "R11" V 4750 850 50  0000 C CNN
-F 1 "1.25k" V 4850 850 50  0000 C CNN
-F 2 "Resistor_SMD:R_0805_2012Metric_Pad1.20x1.40mm_HandSolder" V 4580 850 50  0001 C CNN
-F 3 "~" H 4650 850 50  0001 C CNN
-F 4 "https://www.mouser.de/ProductDetail/Panasonic/ERJ-6ENF1201V?qs=sGAEpiMZZMtG0KNrPCHnjTg0x5DoQJ5PdamLOtzjzkA%3D" H 4650 850 50  0001 C CNN "order"
-	1    4650 850
-	0    1    1    0
-$EndComp
-$Comp
-L power:GND #PWR023
-U 1 1 616ABB8E
-P 4950 850
-F 0 "#PWR023" H 4950 600 50  0001 C CNN
-F 1 "GND" V 4955 722 50  0000 R CNN
-F 2 "" H 4950 850 50  0001 C CNN
-F 3 "" H 4950 850 50  0001 C CNN
-	1    4950 850
 	0    -1   -1   0
 $EndComp
 Wire Wire Line
-	4950 850  4800 850
+	4950 950  4800 950
 $Comp
 L Connector:Conn_01x02_Male J2
@@
 	3450 5800 3950 5800
 Wire Wire Line
-	4950 950  4500 950
+	4950 850  4500 850
 $Comp
 L Connector:TestPoint TP1
@@
 Wire Wire Line
 	3100 3250 3100 3550
+$Comp
+L Device:R R11
+U 1 1 616A8084
+P 4650 950
+F 0 "R11" V 4750 950 50  0000 C CNN
+F 1 "1.25k" V 4850 950 50  0000 C CNN
+F 2 "Resistor_SMD:R_0805_2012Metric_Pad1.20x1.40mm_HandSolder" V 4580 950 50  0001 C CNN
+F 3 "~" H 4650 950 50  0001 C CNN
+F 4 "https://www.mouser.de/ProductDetail/Panasonic/ERJ-6ENF1201V?qs=sGAEpiMZZMtG0KNrPCHnjTg0x5DoQJ5PdamLOtzjzkA%3D" H 4650 950 50  0001 C CNN "order"
+	1    4650 950
+	0    1    1    0
+$EndComp
 $EndSCHEMATC

Commit message: - update 1.25k resistors to 1.2k resistors
Parts:
- R10, R11, R13, R9: value 1.25k -> 1.2k
Changed lines of the file:
@@
 P 5000 5650
 F 0 "R13" H 5070 5696 50  0000 L CNN
-F 1 "1.25k" H 5070 5605 50  0000 L CNN
+F 1 "1.2k" H 5070 5605 50  0000 L CNN
 F 2 "Resistor_SMD:R_0805_2012Metric_Pad1.20x1.40mm_HandSolder" V 4930 5650 50  0001 C CNN
 F 3 "~" H 5000 5650 50  0001 C CNN
@@
 P 3700 3100
 F 0 "R9" V 3493 3100 50  0000 C CNN
-F 1 "1.25k" V 3584 3100 50  0000 C CNN
+F 1 "1.2k" V 3584 3100 50  0000 C CNN
 F 2 "Resistor_SMD:R_0805_2012Metric_Pad1.20x1.40mm_HandSolder" V 3630 3100 50  0001 C CNN
 F 3 "~" H 3700 3100 50  0001 C CNN
@@
 P 3700 3550
 F 0 "R10" V 3493 3550 50  0000 C CNN
-F 1 "1.25k" V 3584 3550 50  0000 C CNN
+F 1 "1.2k" V 3584 3550 50  0000 C CNN
 F 2 "Resistor_SMD:R_0805_2012Metric_Pad1.20x1.40mm_HandSolder" V 3630 3550 50  0001 C CNN
 F 3 "~" H 3700 3550 50  0001 C CNN
@@
 U 1 1 61649099
 P 1650 5250
-F 0 "C1" H 1768 5296 50  0000 L CNN
-F 1 "4.7u" H 1768 5205 50  0000 L CNN
+F 0 "C1" H 1532 5204 50  0000 R CNN
+F 1 "4.7u" H 1532 5295 50  0000 R CNN
 F 2 "Capacitor_SMD:C_0805_2012Metric_Pad1.18x1.45mm_HandSolder" H 1688 5100 50  0001 C CNN
 F 3 "https://www.mouser.de/datasheet/2/427/VISH_S_A0012037911_1-2572454.pdf" H 1650 5250 50  0001 C CNN
 	1    1650 5250
-	1    0    0    -1
+	-1   0    0    1
 $EndComp
 $Comp
@@
 P 4650 950
 F 0 "R11" V 4750 950 50  0000 C CNN
-F 1 "1.25k" V 4850 950 50  0000 C CNN
+F 1 "1.2k" V 4850 950 50  0000 C CNN
 F 2 "Resistor_SMD:R_0805_2012Metric_Pad1.20x1.40mm_HandSolder" V 4580 950 50  0001 C CNN
 F 3 "~" H 4650 950 50  0001 C CNN
